File: PCB/Tiny4FSK.kicad_sch (KiCad schematic)
At the start: 68 parts, among them IC1 SI4063, J1 I2C, J2 USBC, J3 SPI, J4 JTAG, J5 PWR Batt, J6 PWR Supply, SW1 RST, SW2 SOURCE, SW3 BATT PWR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

Commit message: Update Tiny4FSK.kicad_sch
Parts:
- added JP1: SWITCH_EN, Jumper:SolderJumper-2_P1.3mm_Open_Pad1.0x1.5mm, symbol Jumper:Jumper_2_Open
- SW2: footprint SlideSwitch:WS-SLSU_6p7x2p7_WRE -> Jumper:SolderJumper-3_P1.3mm_Open_Pad1.0x1.5mm
Connections:
- net +BATT: now also JP1.2 (B)
- net BST_IN: now also JP1.1 (A)
- net Earth: now also J4.3 (Pin_3), J4.5 (Pin_5)
Changed lines of the file:
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@@
   (junction (at 210.312 80.264) (diameter 0) (color 0 0 0 0)
   )
+  (junction (at 146.812 172.466) (diameter 0) (color 0 0 0 0)
+  )
   (junction (at 136.398 64.516) (diameter 0) (color 0 0 0 0)
   )
@@
   (junction (at 161.544 39.37) (diameter 0) (color 0 0 0 0)
   )
+  (junction (at 68.0979 163.83) (diameter 0) (color 0 0 0 0)
+  )
   (junction (at 109.474 23.368) (diameter 0) (color 0 0 0 0)
   )
@@
     (stroke (width 0) (type default))
   )
+  (wire (pts (xy 136.652 164.846) (xy 146.812 164.846))
+    (stroke (width 0) (type default))
+  )
   (wire (pts (xy 120.142 23.368) (xy 120.142 34.544))
     (stroke (width 0) (type default))
@@
     (stroke (width 0) (type default))
   )
+  (wire (pts (xy 68.0979 163.83) (xy 77.47 163.83))
+    (stroke (width 0) (type default))
+  )
   (wire (pts (xy 231.4213 79.756) (xy 231.394 79.756))
     (stroke (width 0) (type default))
@@
     (stroke (width 0) (type default))
   )
-  (wire (pts (xy 68.072 163.83) (xy 77.47 163.83))
+  (wire (pts (xy 68.072 163.83) (xy 68.0979 163.83))
     (stroke (width 0) (type default))
   )
@@
     (stroke (width 0) (type default))
   )
+  (wire (pts (xy 146.812 164.846) (xy 146.812 172.466))
+    (stroke (width 0) (type default))
+  )
   (wire (pts (xy 121.92 131.572) (xy 122.174 131.572))
     (stroke (width 0) (type default))
@@
       (effects (font (size 1.27 1.27)))
     )
-    (property "Footprint" "SlideSwitch:WS-SLSU_6p7x2p7_WRE" (at 142.494 158.115 0)
+    (property "Footprint" "Jumper:SolderJumper-3_P1.3mm_Open_Pad1.0x1.5mm" (at 142.494 158.115 0)
       (effects (font (size 1.27 1.27)) hide)
     )
@@
     )
   )
+  (symbol (lib_id "Jumper:Jumper_2_Open") (at 136.652 169.926 90) (unit 1)
+    (in_bom yes) (on_board yes) (dnp no)
+    (property "Reference" "JP1" (at 126.746 165.735 90)
+      (effects (font (size 1.27 1.27)) (justify right))
+    )
+    (property "Value" "SWITCH_EN" (at 125.476 172.466 90)
+      (effects (font (size 1.27 1.27)) (justify right))
+    )
+    (property "Footprint" "Jumper:SolderJumper-2_P1.3mm_Open_Pad1.0x1.5mm" (at 136.652 169.926 0)
+      (effects (font (size 1.27 1.27)) hide)
+    )
+    (property "Datasheet" "~" (at 136.652 169.926 0)
+      (effects (font (size 1.27 1.27)) hide)
+    )
+    (pin "1")
+    (pin "2")
+    (instances
+      (project "Tiny4FSK"
+        (path "/afd8b0bc-328a-481f-8ddf-c1252dc3b440"
+          (reference "JP1") (unit 1)
+        )
+      )
+    )
+  )
   (symbol (lib_id "Device:R_Small_US") (at 150.368 106.426 270) (unit 1)
     (in_bom yes) (on_board yes) (dnp no) (fields_autoplaced)
@@
     )
   )
+  (symbol (lib_name "Earth_2") (lib_id "power:Earth") (at 68.0979 163.83 0) (mirror y) (unit 1)
+    (in_bom yes) (on_board yes) (dnp no) (fields_autoplaced)
+    (property "Reference" "#PWR049" (at 68.0979 170.18 0)
+      (effects (font (size 1.27 1.27)) hide)
+    )
+    (property "Value" "Earth" (at 68.0979 167.64 0)
+      (effects (font (size 1.27 1.27)) hide)
+    )
+    (property "Footprint" "" (at 68.0979 163.83 0)
+      (effects (font (size 1.27 1.27)) hide)
+    )
+    (property "Datasheet" "~" (at 68.0979 163.83 0)
+      (effects (font (size 1.27 1.27)) hide)
+    )
+    (pin "1")
+    (instances
+      (project "Tiny4FSK"
+        (path "/afd8b0bc-328a-481f-8ddf-c1252dc3b440"
+          (reference "#PWR049") (unit 1)
+        )
+      )
+    )
+  )
   (symbol (lib_name "+BATT_1") (lib_id "power:+BATT") (at 149.606 172.466 0) (unit 1)
     (in_bom yes) (on_board yes) (dnp no) (fields_autoplaced)
@@
   )
   (symbol (lib_id "Switch:SW_SPDT") (at 141.732 175.006 0) (unit 1)
-    (in_bom yes) (on_board yes) (dnp no) (fields_autoplaced)
-    (property "Reference" "SW3" (at 141.732 167.64 0)
+    (in_bom yes) (on_board yes) (dnp no)
+    (property "Reference" "SW3" (at 139.065 177.927 0)
       (effects (font (size 1.27 1.27)))
     )
-    (property "Value" "BATT PWR" (at 141.732 170.18 0)
+    (property "Value" "BATT PWR" (at 139.065 180.467 0)
       (effects (font (size 1.27 1.27)))
     )
