File: PCB/Tiny4FSK.kicad_pcb (KiCad board)
At the start: 4 copper layers, 30.9 x 66 mm, 70 parts, among them IC1 SI4063, J1 I2C, J2 USBC, J3 SPI, J4 JTAG, J5 PWR Batt, J6 PWR Supply, SW1 RST, SW2 SOURCE, SW3 BATT PWR, U1 BME280, U2 MAX-M10S, U3 ATSAMD21G18A-A, U4 Linear Step-Down, U5 TPS61200DRC

Commit message: Update Tiny4FSK.kicad_pcb
Parts:
- removed REF** (x2): MountingHole_2.2mm_M2, MountingHole:MountingHole_2.2mm_M2
- added JP1: SWITCH_EN, Jumper:SolderJumper-2_P1.3mm_Open_Pad1.0x1.5mm, F.Cu at (154.0, 123.3)
- AE2: footprint Ant:Antenna_Whip -> Antenna:Antenna_Whip
- SW2: footprint SlideSwitch:WS-SLSU_6p7x2p7_WRE -> Jumper:SolderJumper-3_P1.3mm_Open_Pad1.0x1.5mm
- moved C19 39.4 mm to (152.4, 115.7), turned to -90 degrees
- moved XTAL2 37.7 mm to (156.6, 119.9)
- moved C14 37.1 mm to (153.1, 119.5), turned to 180 degrees
- moved C26 36.6 mm to (164.4, 115.0)
- moved AE1 36.6 mm to (164.3, 64.7)
- moved BT1 36.6 mm to (148.2, 119.5)
- moved C1 36.6 mm to (142.9, 84.5)
- moved C10 36.6 mm to (142.8, 103.6)
- moved C11 36.6 mm to (139.0, 88.1)
- moved C12 36.6 mm to (154.6, 96.9)
- moved C13 36.6 mm to (164.7, 97.7)
- moved C15 36.6 mm to (144.1, 122.2)
- moved C16 36.6 mm to (148.2, 112.0)
- moved C17 36.6 mm to (144.4, 114.3)
- moved C2 36.6 mm to (150.5, 85.1)
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Connections:
- J4 pad 3: Net-(J2-Pin_3) -> Earth
- J4 pad 5: Net-(J2-Pin_3) -> Earth
Routing:
- net RF_RST: track 21.0 -> 10.2 mm, vias 2 -> 3
- net Earth: track 123.6 -> 134.1 mm, vias 138 -> 126
- net BATT_SENSE: track 64.8 -> 73.5 mm, vias 5 -> 6
- net SCK: track 21.5 -> 25.1 mm
- net Net-(J2-Pin_3): track 2.57 -> 0.00 mm
- net MOSI: track 36.9 -> 34.5 mm
- net LIN: track 50.6 -> 52.7 mm
- net GPIO1: track 8.89 -> 10.9 mm
- net +3.3V: track 61.7 -> 63.7 mm, vias 16 -> 17
- net GPIO0: track 13.0 -> 14.9 mm
- net MISO: track 27.6 -> 29.5 mm
- net BST_IN: track 41.6 -> 43.2 mm
- net RF_SS: track 21.9 -> 23.1 mm
- net BOOST: track 21.2 -> 22.3 mm
- added copper zone on F.Cu, net LIN
Other:
- board text added: "3V3"
- board text added: "3V3 GND"
- board text added: "3V3 SDA SCL GND"
- board text added: "GND SCK MISO MOSI 3V3"
- board text added: "RST"
- board text added: "SW CTRL"
- board text added: "UNREG GND"
- board text added: "USB BATT"

Commit message: Update Tiny4FSK.kicad_pcb
Parts:
- removed the J4 at (167.8, 97.9)
- removed the J5 at (167.8, 87.7)
- removed the SW2 at (144.4, 128.0)
- removed the XTAL1 at (152.2, 102.3)
- added C7: 100 pF, Capacitor_SMD:C_0805_2012Metric_Pad1.18x1.45mm_HandSolder, F.Cu at (151.0, 99.8)
- added D3: Power, LED_SMD:LED_0805_2012Metric_Pad1.15x1.40mm_HandSolder, F.Cu at (139.2, 128.8)
- added G***: LOGO, LOGO, F.Cu at (451.5, 114.2)
- added G***: LOGO, LOGO, B.Cu at (142.5, 127.5)
- added H1: MountingHole, MountingHole:MountingHole_2.2mm_M2, F.Cu at (157.2, 74.5)
- added H2: MountingHole, MountingHole:MountingHole_2.2mm_M2, F.Cu at (163.8, 93.8)
- added H3: MountingHole, MountingHole:MountingHole_2.2mm_M2, F.Cu at (159.2, 124.2)
- added H4: MountingHole, MountingHole:MountingHole_2.2mm_M2, F.Cu at (140.0, 122.8)
- added J1: SWD, Connector_PinHeader_2.54mm:PinHeader_1x06_P2.54mm_Vertical, F.Cu at (140.2, 74.8)
- added J2: OPTIONAL, Jumper:SolderJumper-2_P1.3mm_Open_Pad1.0x1.5mm, F.Cu at (151.5, 97.5)
- added JP2: Source, Jumper:SolderJumper-3_P1.3mm_Open_Pad1.0x1.5mm_NumberLabels, F.Cu at (144.4, 128.2)
- added U4: TCXO MCU, Oscillator_TCXO:ATXK-H11-E-32.768KHZ-E50-T3, F.Cu at (150.9, 109.2)
- J4: renamed from J3; footprint Connector_PinHeader_1.00mm:PinHeader_1x05_P1.00mm_Vertical -> Connector_PinHeader_2.54mm:PinHeader_1x05_P2.54mm_Vertical
- J5: renamed from J1; footprint Connector_PinHeader_1.00mm:PinHeader_1x04_P1.00mm_Vertical -> Connector_PinHeader_2.54mm:PinHeader_1x04_P2.54mm_Vertical
- J6: value PWR Supply -> Power; footprint Connector_PinHeader_1.00mm:PinHeader_1x02_P1.00mm_Vertical -> Connector_PinHeader_2.54mm:PinHeader_1x03_P2.54mm_Vertical
- R11: value 10k -> 900k
- R12: value 56k -> 5M
- XTAL1: renamed from XTAL2; footprint TCXO:ECSTXO20CSMV4384AYTR -> OSC:OSC_ECS-TXO-32CSMV-260-AN-TR
- moved J5 16.3 mm to (167.8, 100.8)
- moved J6 9.23 mm to (167.8, 104.6), turned to 0 degrees
- moved J4 4.13 mm to (167.8, 113.4)
- moved R3 1.55 mm to (147.7, 100.7), turned to 90 degrees
- moved C5 0.95 mm to (163.8, 97.5)
- moved C21 0.95 mm to (152.3, 114.8)
- moved R7 0.89 mm to (164.8, 102.6)
- moved C25 0.80 mm to (152.6, 118.9)
- moved R8 0.69 mm to (164.0, 99.8)
- moved SW2 0.42 mm to (153.1, 129.2)
- moved BT1 0.34 mm to (148.2, 119.2)
- moved XTAL1 0.33 mm to (156.3, 120.0)
- renumbered C11 to C1, C7 to C10, C8 to C11, C9 to C12, C10 to C13, C16 to C14, C12 to C15, C5 to C16, C25 to C17, C17 to C18, C23 to C19, C18 to C20, C19 to C21, C21 to C22, C15 to C23, C14 to C25, C22 to C27, C4 to C3, C1 to C4, C13 to C5, C20 to C8, C3 to C9, J2 to J3, L6 to L2, L2 to L3, L3 to L4, L4 to L6, R3 to R10, R6 to R3, R7 to R6, R10 to R7, R9 to R8, R8 to R9, SW3 to SW2, U2 to U1, U1 to U2, U4 to U3, U3 to U5, U5 to U6
Connections:
- C4 pad 1: +3.3V -> LDO
- IC1 pad 1: unconnected-(IC1-SDN-Pad1) -> SDN
- J6 pad 1: +3.3V -> BATT_SENSE
- U3 pad 2: +3.3V -> LIN
- U3 pad 3: LIN -> LDO
- U5 pad 1: Net-(U3-PA00) -> TCXO
- U5 pad 2: unconnected-(U3-PA01-Pad2) -> OPT XOUT
- U5 pad 25: unconnected-(U3-PA16-Pad25) -> SDN
Routing:
- net LDO: track 0.00 -> 51.5 mm, vias 0 -> 3
- net LIN: track 52.7 -> 11.5 mm, vias 2 -> 0
- net SWCLK: track 12.8 -> 36.0 mm
- net SCK: track 25.1 -> 45.1 mm, vias 2 -> 3
- net SWDIO: track 20.4 -> 35.0 mm, vias 2 -> 1
- net nRST: track 54.9 -> 43.3 mm, vias 4 -> 3
- net MISO: track 29.5 -> 40.5 mm, vias 2 -> 4
- net SDN: track 0.00 -> 10.9 mm, vias 0 -> 2
- net Earth: track 134.1 -> 123.6 mm, vias 126 -> 172
- net TCXO: track 0.00 -> 7.40 mm
- net SCL: track 44.1 -> 51.3 mm
- net OPT XOUT: track 0.00 -> 6.74 mm
- net EXTINT: track 22.2 -> 28.1 mm
- net MOSI: track 34.5 -> 38.8 mm
- net BATT_SENSE: track 73.5 -> 69.4 mm, vias 6 -> 5
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- added copper zone on F.Cu, net Earth
Other:
- board size 30.9 x 66 mm -> 30.9 x 65.8 mm
- board text added: "3v3"
- board text added: "JP1 - Control PWR source (USB and CTR for USB, CTR and BATT) JP2 - Cut to enable SW2 for PWR SW1 - RST SW2 - BATT PWR AE2 - 70cm ANT"
- board text added: "Rev. 2 - 3/13/24"
- board text removed: "3V3"
- board text removed: "3V3 GND"
- board text removed: "3V3 SDA SCL GND"
- board text removed: "GND SCK MISO MOSI 3V3"
- board text removed: "UNREG GND"
