File: PCB + Schematic/Rev. 4/_autosave-Tiny4FSK.kicad_pcb (KiCad board)
At the start: 4 copper layers, 35.3 x 73.6 mm, 84 parts, among them J1 Power Ext, J2 GPIO, J3 I2C, J4 USB, J5 USB Breakout, J6 SPI, J7 USBC, J8 SWD, SW1 Power Switch, SW2 RST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

Commit message: Matching on GPS, modifications
Parts:
- added G***: LOGO, LOGO, B.Cu at (144.7, 43.1)
- moved G*** 6.58 mm to (159.3, 41.5)
- moved G*** 5.13 mm to (144.4, 41.0)
- moved G*** 0.51 mm to (149.1, 80.1)
- moved G*** 0.10 mm to (149.1, 67.5)
Routing:
- net +3.3V: track 76.3 -> 78.8 mm
- net Earth: track 41.1 -> 42.1 mm, vias 137 -> 136
Other:
- board text added: "3v3"
- board text added: "A1"
- board text added: "A2"
- board text added: "D12"
- board text added: "D13"
- board text added: "GND"
- board text added: "MISO"
- board text added: "MOSI"
- board text added: "November 2024"
- board text added: "Rev. 4.0"
- board text added: "SCK"
- board text added: "SCL"
- board text added: "SDA"
- board text added: "Sponsored by:"
- board text removed: "October 15, 2024"
- board text removed: "Rev. 2.0"
