File: PCB + Schematic/Rev. 4/Tiny4FSK.kicad_sch (KiCad schematic)
At the start: 79 parts, among them J1 SWD, J2 GPIO, J3 USBC, J4 USB, J5 I2C, J6 Power Ext, J7 SPI, J8 USB Breakout, SW1 RST, SW2 Power Switch, U1 ATSAMD21G18A-A, U2 ATGM336H, U2 TPS61200DRC, U3 SI4063, U5 1XZA032768AD19, U8 Linear Step-Down

Commit message: JLCPCB export, Silkscreen
Parts:
- renumbered C28 to C1, C11 to C13, C19 to C15, C20 to C16, C4 to C17, C6 to C18, C1 to C19, C22 to C20, C23 to C21, C5 to C22, C18 to C23, C25 to C24, C3 to C25, J6 to J1, J5 to J3, J8 to J5, J7 to J6, J3 to J7, J1 to J8, R2 to R1, R7 to R10, R3 to R11, R5 to R12, R10 to R13, R13 to R14, R9 to R15, R1 to R2, R12 to R3, R11 to R4, R14 to R5, R15 to R6, R4 to R7, R6 to R8, R8 to R9, SW2 to SW1, U5 to U4, U3 to U6, U8 to U7, U7 to U8

Commit message: LNA Add-On, Silkscreen
Parts:
- added AE3: GPS1003, RF_Antenna_Extended:GPS1003, symbol Device:Antenna
- added C28: 100nF, Capacitor_SMD:C_0402_1005Metric_Pad0.74x0.62mm_HandSolder, symbol Device:C_Small
- added C29: 470 pF, Capacitor_SMD:C_0402_1005Metric_Pad0.74x0.62mm_HandSolder, symbol Device:C_Small
- added L8: 6.8 nH, Inductor_SMD:L_0402_1005Metric_Pad0.77x0.64mm_HandSolder, symbol Device:L
- added U9: ~, Package_DFN_QFN:DFN-6-1EP_2x2mm_P0.65mm_EP1x1.6mm, symbol LNA:AT2659
Connections:
- net +3.3V: now also C28.2, U9.4 (VCC), U9.5 (SHDN)
- net Earth: now also C28.1, U9.1 (GND), U9.2 (GND)
- new net: L8.2, U9.3 (RFIN)
- new net: C29.1, L8.1
- new net: AE3.1 (A), C29.2
- new net RFOUT: U9.6 (RFOUT)

Commit message: LNA Addon, JLC Parts
Parts:
- added U10: ~, AddOns:LNA_AddOn, symbol AddOns:LNA_AddOn
- AE3: now not fitted
- C29: footprint Capacitor_SMD:C_0402_1005Metric_Pad0.74x0.62mm_HandSolder -> Capacitor_SMD:C_0603_1608Metric_Pad1.08x0.95mm_HandSolder; LCSC C52923 -> C1620
- L8: LCSC C307609 -> C108260
- U9: LCSC (none) -> C92450
Connections:
- net +3.3V: now also U10.4 (3v3)
- net Earth: now also U10.3 (GND)
- net RFOUT: now also U10.1 (RFOUT)

Commit message: LNA, JLCPCB
Parts:
- U9: footprint Package_DFN_QFN:DFN-6-1EP_2x2mm_P0.65mm_EP1x1.6mm -> LDO:DFN-6_L1.6-W1.0-P0.55-BL
Changed lines of the file:
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@@
 			)
 		)
-		(property "Footprint" "Package_DFN_QFN:DFN-6-1EP_2x2mm_P0.65mm_EP1x1.6mm"
+		(property "Footprint" "LDO:DFN-6_L1.6-W1.0-P0.55-BL"
 			(at 136.144 164.846 0)
 			(effects

Commit message: PCB Layout, RF Matching
Parts:
- removed AE3: GPS1003, RF_Antenna_Extended:GPS1003, symbol Device:Antenna
- removed C28: 100nF, Capacitor_SMD:C_0402_1005Metric_Pad0.74x0.62mm_HandSolder, symbol Device:C_Small
- removed C29: 470 pF, Capacitor_SMD:C_0603_1608Metric_Pad1.08x0.95mm_HandSolder, symbol Device:C_Small
- removed L8: 6.8 nH, Inductor_SMD:L_0402_1005Metric_Pad0.77x0.64mm_HandSolder, symbol Device:L
- removed U10: ~, AddOns:LNA_AddOn, symbol AddOns:LNA_AddOn
- removed U9: ~, LDO:DFN-6_L1.6-W1.0-P0.55-BL, symbol LNA:AT2659
- C20: value 15 pF -> 8 pF
- C24: value 12 pF -> 6 pF
- C27: value 10 pF -> 5 pF
- L4: value 33 nH -> 14 nH
- L5: value 30 nH -> 14 nH
- L6: value 36 nH -> 14 nH
- L7: value 22 nH -> 14 nH

Commit message: Matching on GPS, modifications
Parts:
- removed C13: 100 pF, Capacitor_SMD:C_0402_1005Metric_Pad0.74x0.62mm_HandSolder, symbol Device:C_Small
- added C28: 1.5pF, Capacitor_SMD:C_0402_1005Metric_Pad0.74x0.62mm_HandSolder, symbol Device:C_Small
- added L8: 3.9 nH, Inductor_SMD:L_0402_1005Metric_Pad0.77x0.64mm_HandSolder, symbol Device:L
- AE1: value GPS1003 -> 1575AT43A0040; footprint RF_Antenna_Extended:GPS1003 -> RF_Antenna_Extended:ANT_1575AT_JOT
- C1, C14: footprint Capacitor_SMD:C_0603_1608Metric_Pad1.08x0.95mm_HandSolder -> Capacitor_SMD:C_0402_1005Metric_Pad0.74x0.62mm_HandSolder
- C19: value 4.5 nF -> 4.7 nF; footprint Capacitor_SMD:C_0805_2012Metric_Pad1.18x1.45mm_HandSolder -> Capacitor_SMD:C_0402_1005Metric_Pad0.74x0.62mm_HandSolder
- L1: value 33 nH -> 3.9 nH
- R10, R12: footprint Resistor_SMD:R_0805_2012Metric_Pad1.20x1.40mm_HandSolder -> Resistor_SMD:R_0402_1005Metric_Pad0.72x0.64mm_HandSolder
- R13, R14, R15, R8, R9: footprint Resistor_SMD:R_0603_1608Metric_Pad0.98x0.95mm_HandSolder -> Resistor_SMD:R_0402_1005Metric_Pad0.72x0.64mm_HandSolder
- SW1: footprint Button_Switch_SMD:SW_SPST_CK_RS282G05A3 -> Button_Switch_SMD:SW_Tactile_SPST_NO_Straight_CK_PTS636Sx25SMTRLFS
Connections:
- net ANT_GPS: now also C28.1, L8.2; no longer AE1.1 (A), L1.2
- net Earth: now also L8.1
- net TCXO: now also U4.3 (OUTPUT)
- new net: AE1.1 (A), C28.2, L1.2
Other:
- note added: "Look into: SXBP-425+"
- moved on the sheet: AE1, C1, L1, U2

Commit message: Finished?
Parts:
- U4: value 1XZA032768AD19 -> ECS-327TXO-2012; footprint Oscillator_TCXO:KDS-1XZA032768AD19 -> Oscillator_TCXO:ECS-327TXO-2012
- U8: footprint OSC:OSC_ECS-TXO-32CSMV-260-AN-TR -> Oscillator_TCXO:ECS-TXO-20CSMV4
Changed lines of the file:
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@@
 			)
 		)
-		(property "Value" "1XZA032768AD19"
+		(property "Value" "ECS-327TXO-2012"
 			(at 247.65 118.364 0)
 			(effects
@@
 			)
 		)
-		(property "Footprint" "Oscillator_TCXO:KDS-1XZA032768AD19"
+		(property "Footprint" "Oscillator_TCXO:ECS-327TXO-2012"
 			(at 247.65 118.11 0)
 			(effects
@@
 			)
 		)
-		(property "Footprint" "OSC:OSC_ECS-TXO-32CSMV-260-AN-TR"
+		(property "Footprint" "Oscillator_TCXO:ECS-TXO-20CSMV4"
 			(at 38.354 130.048 0)
 			(effects

Commit message: 3d models
Parts:
- U6: now fitted
Changed lines of the file:
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@@
 		(in_bom yes)
 		(on_board yes)
-		(dnp yes)
+		(dnp no)
 		(fields_autoplaced yes)
 		(property "Reference" "U6"
