File: PCB + Schematic/Tiny4FSK.kicad_sch (KiCad schematic)
At the start: 83 parts, among them J1 Power Ext, J2 GPIO, J3 I2C, J4 USB, J5 USB Breakout, J6 SPI, J7 USBC, J8 SWD, J9 Counterpoise, SW1 Power Switch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

Commit message: kicad 10!
Parts:
- U8: value ~ -> (none)

Commit message: new batch pcb
Parts:
- C28: value 1.5pF -> 2.7pF
Changed lines of the file:
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@@
 			)
 		)
-		(property "Value" "1.5pF"
+		(property "Value" "2.7pF"
 			(at 74.93 80.5115 0)
 			(show_name no)
