File: PCB + Schematic/Tiny4FSK.kicad_pcb (KiCad board)
At the start: 4 copper layers, 35.1 x 76.3 mm, 90 parts, among them J1 Power Ext, J2 GPIO, J3 I2C, J4 USB, J5 USB Breakout, J6 SPI, J7 USBC, J8 SWD, J9 Counterpoise, SW1 Power Switch, SW2 RST, U1 BME280, U2 ATGM336H, U3 TPS61200DRC, U4 ECS-327TXO-2012, U5 ATSAMD21G18A-A, U6 SI4063, U7 Linear Step-Down

Commit message: kicad 10 (not nightly)
Parts:
- C28: value 1.5pF -> 2.7pF
