File: hardware/Tiny4FSK.kicad_sch (KiCad schematic)
At the start: 0 parts

Commit message: first new schem rev
Changed lines of the file:
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@@
 	)
 	(sheet
-		(at 67.31 86.36)
-		(size 21.59 15.24)
+		(at 67.31 83.82)
+		(size 21.59 17.78)
 		(exclude_from_sim no)
 		(in_bom yes)
@@
 		)
 		(property "Sheetname" "sensors"
-			(at 67.31 85.6484 0)
+			(at 67.31 83.1084 0)
 			(show_name no)
 			(do_not_autoplace no)
