File: hardware/power.kicad_sch (KiCad schematic)
At the start: 27 parts, among them J7 GCT-4105, SW1 PWR, U10 USBLC6-2SC6, U3 TPS61200DRC, U7 XC6210B332MR, U9 TPS2116DRL

Commit message: more placement
Connections:
- net RAW.D+: now reaches J7.A6 (D+), J7.B6 (D+), U10.3 (I/O2)
- net RAW.D-: now reaches J7.A7 (D-), J7.B7 (D-), U10.1 (I/O1)
Changed lines of the file:
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@@
+		)
+	)
+	(label "RAW.D+"
+		(at 58.42 67.31 0)
+		(effects
+			(font
+				(size 1.27 1.27)
+			)
+			(justify left bottom)
+		)
+	)
+	(label "RAW.D-"
+		(at 58.42 64.77 0)
+		(effects
+			(font
+				(size 1.27 1.27)
+			)
+			(justify left bottom)
 		)
 	)
