File: hardware/interface.kicad_sch (KiCad schematic)
At the start: 16 parts, among them J1 EXT_PWR, J2 GPIO, J3 I2C, J4 USB, J6 SPI, J8 SWD

Commit message: first new schem rev
Parts:
- J8: footprint Connector_PinHeader_1.27mm:PinHeader_2x05_P1.27mm_Vertical_SMD -> Connector_Pogo_1.27mm:Pogo_2x05_P1.27mm
Other:
- note removed: "POGO: 1.17mm"
- note removed: "TODO: MAKE COMPT. WITH POGO PIN"
- moved on the sheet: J1, J2, J3, J4, J6, J8

Commit message: pcb rework -- layout subsections and rough floorplanning
Parts:
- D1, D2, D3: footprint LED_SMD:LED_0805_2012Metric_Pad1.15x1.40mm_HandSolder -> LED_SMD:LED_0603_1608Metric
- R13, R15: value 330 -> 330R; footprint Resistor_SMD:R_0402_1005Metric_Pad0.72x0.64mm_HandSolder -> Capacitor_SMD:C_0402_1005Metric
- R14: footprint Resistor_SMD:R_0402_1005Metric_Pad0.72x0.64mm_HandSolder -> Capacitor_SMD:C_0402_1005Metric
Connections:
- net Earth: now also D1.1 (K), D2.1 (K), D3.1 (K); no longer R13.2, R14.2, R15.2
- net LED.ERROR: now also R15.1; no longer D1.2 (A)
- net LED.SUCCESS: now also R13.1; no longer D2.2 (A)
- net at R14.1: now also JP2.1 (A); no longer D3.1 (K)
- net at D3.2 (A): now also R14.2; no longer JP2.1 (A)
- new net: D1.2 (A), R15.2
- new net: D2.2 (A), R13.2
Other:
- moved on the sheet: D1, D2, D3, R13, R14, R15

Commit message: lay out programming header + button, move powerpath near tx
Other:
- note added: "COMBINE INTO SHIELD LAYOUT MORE VCC PINS"
Changed lines of the file:
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@@
 	(generator_version "10.0")
 	(paper "A4")
+	(text "COMBINE INTO SHIELD LAYOUT\n\nMORE VCC PINS"
+		(exclude_from_sim no)
+		(at 175.514 37.846 0)
+		(effects
+			(font
+				(size 1.27 1.27)
+			)
+		)
+	)
 	(junction
 		(at 186.69 62.23)

Commit message: draft of gpio layout
Parts:
- removed J1: EXT_PWR, Connector_PinHeader_2.54mm:PinHeader_1x03_P2.54mm_Vertical, symbol Connector_Generic:Conn_01x03
- removed J2: GPIO, Connector_PinHeader_2.54mm:PinHeader_1x09_P2.54mm_Vertical, symbol Connector_Generic:Conn_01x09
- removed J3: I2C, Connector_PinHeader_2.54mm:PinHeader_1x04_P2.54mm_Vertical, symbol Connector_Generic:Conn_01x04
- removed J4: USB, Connector_PinHeader_2.54mm:PinHeader_1x04_P2.54mm_Vertical, symbol Connector_Generic:Conn_01x04
- removed J6: SPI, Connector_PinHeader_2.54mm:PinHeader_1x05_P2.54mm_Vertical, symbol Connector_Generic:Conn_01x05
- added J10: GPIO_ROW, Connector_PinHeader_2.54mm:PinHeader_1x15_P2.54mm_Vertical, symbol Connector_Generic:Conn_01x15
- added J2: PWR, Connector_PinHeader_2.54mm:PinHeader_1x06_P2.54mm_Vertical, symbol Connector_Generic:Conn_01x06
Connections:
- net +3.3V: now also J2.4 (Pin_4), J2.6 (Pin_6)
- net +BATT: now also J2.2 (Pin_2)
- net Earth: now also J10.1 (Pin_1), J10.12 (Pin_12), J10.15 (Pin_15), J10.4 (Pin_4), J10.8 (Pin_8), J2.1 (Pin_1), J2.3 (Pin_3), J2.5 (Pin_5)
- net GP.CLK: now also J10.7 (Pin_7)
- net GP.GPIO12: now also J10.9 (Pin_9)
- net GP.GPIO13: now also J10.10 (Pin_10)
- net GP.GPIO38: now also J10.11 (Pin_11)
- net GP.GPIO_A_1: now also J10.13 (Pin_13)
- net GP.GPIO_A_2: now also J10.14 (Pin_14)
- net GP.MISO: now also J10.6 (Pin_6)
- net GP.MOSI: now also J10.5 (Pin_5)
- net GP.SCL: now also J10.3 (Pin_3)
- net GP.SDA: now also J10.2 (Pin_2)

Commit message: net class shenanigans
Parts:
- D1, D2, D3, R13, R14, R15: KiLib_Generator (none) -> SMD_2terminal_chip_molded
- H1, H2, H4: KiLib_Generator (none) -> mounting_hardware/mounting_hole
- J10, J2: KiLib_Generator (none) -> connector/pin_header_socket
Changed lines of the file:
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@@
+			)
+		)
+		(property "KiLib_Generator" "SMD_2terminal_chip_molded"
+			(at 86.36 125.73 0)
+			(hide yes)
+			(show_name no)
+			(do_not_autoplace no)
+			(effects
+				(font
+					(size 1.27 1.27)
+				)
 			)
 		)
@@
 		)
 		(property "Mouser Price/Stock" ""
+			(at 115.57 125.73 0)
+			(hide yes)
+			(show_name no)
+			(do_not_autoplace no)
+			(effects
+				(font
+					(size 1.27 1.27)
+				)
+			)
+		)
+		(property "KiLib_Generator" "SMD_2terminal_chip_molded"
 			(at 115.57 125.73 0)
 			(hide yes)
@@
 			)
 		)
+		(property "KiLib_Generator" "SMD_2terminal_chip_molded"
+			(at 115.57 133.35 0)
+			(hide yes)
+			(show_name no)
+			(do_not_autoplace no)
+			(effects
+				(font
+					(size 1.27 1.27)
+				)
+			)
+		)
 		(pin "1"
 		)
@@
 		(property "Mouser Price/Stock" ""
 			(at 101.6 133.35 90)
+			(hide yes)
+			(show_name no)
+			(do_not_autoplace no)
+			(effects
+				(font
+					(size 1.27 1.27)
+				)
+			)
+		)
+		(property "KiLib_Generator" "SMD_2terminal_chip_molded"
+			(at 101.6 133.35 0)
 			(hide yes)
 			(show_name no)
@@
 			)
 		)
+		(property "KiLib_Generator" "mounting_hardware/mounting_hole"
+			(at 165.1 132.08 0)
+			(hide yes)
+			(show_name no)
+			(do_not_autoplace no)
+			(effects
+				(font
+					(size 1.27 1.27)
+				)
+			)
+		)
 		(instances
 			(project "Tiny4FSK"
@@
 			)
 		)
+		(property "KiLib_Generator" "mounting_hardware/mounting_hole"
+			(at 165.1 119.38 0)
+			(hide yes)
+			(show_name no)
+			(do_not_autoplace no)
+			(effects
+				(font
+					(size 1.27 1.27)
+				)
+			)
+		)
 		(instances
 			(project "Tiny4FSK"
@@
 		)
 		(property "Description" "Generic connector, single row, 01x15, script generated (kicad-library-utils/schlib/autogen/connector/)"
+			(at 210.82 74.93 0)
+			(hide yes)
+			(show_name no)
+			(do_not_autoplace no)
+			(effects
+				(font
+					(size 1.27 1.27)
+				)
+			)
+		)
+		(property "KiLib_Generator" "connector/pin_header_socket"
 			(at 210.82 74.93 0)
 			(hide yes)
@@
 			)
 		)
+		(property "KiLib_Generator" "SMD_2terminal_chip_molded"
+			(at 86.36 133.35 0)
+			(hide yes)
+			(show_name no)
+			(do_not_autoplace no)
+			(effects
+				(font
+					(size 1.27 1.27)
+				)
+			)
+		)
 		(pin "1"
 		)
@@
 		)
 		(property "Mouser Price/Stock" ""
+			(at 101.6 125.73 0)
+			(hide yes)
+			(show_name no)
+			(do_not_autoplace no)
+			(effects
+				(font
+					(size 1.27 1.27)
+				)
+			)
+		)
+		(property "KiLib_Generator" "SMD_2terminal_chip_molded"
 			(at 101.6 125.73 0)
 			(hide yes)
@@
 			)
 		)
+		(property "KiLib_Generator" "mounting_hardware/mounting_hole"
+			(at 165.1 125.73 0)
+			(hide yes)
+			(show_name no)
+			(do_not_autoplace no)
+			(effects
+				(font
+					(size 1.27 1.27)
+				)
+			)
+		)
 		(instances
 			(project "Tiny4FSK"
@@
 			(at 167.64 58.42 0)
 			(hide yes)
+			(show_name no)
+			(do_not_autoplace no)
+			(effects
+				(font
+					(size 1.27 1.27)
+				)
+			)
+		)
+		(property "KiLib_Generator" "connector/pin_header_socket"
+			(at 167.64 58.42 0)
+			(hide yes)

Commit message: draft of routing
Connections:
- net +3.3V: now also J2.2 (Pin_2); no longer J2.6 (Pin_6)
- net +BATT: now also J2.6 (Pin_6); no longer J2.2 (Pin_2)
- net GP.GPIO12: now also J10.11 (Pin_11); no longer J10.9 (Pin_9)
- net GP.GPIO13: now also J10.9 (Pin_9); no longer J10.10 (Pin_10)
- net GP.GPIO38: no longer J10.11 (Pin_11)
- net GP.GPIO_A_1: now also J10.2 (Pin_2); no longer J10.13 (Pin_13)
- net GP.GPIO_A_2: now also J10.3 (Pin_3); no longer J10.14 (Pin_14)
- net GP.SCL: now also J10.13 (Pin_13); no longer J10.3 (Pin_3)
- net GP.SDA: now also J10.14 (Pin_14); no longer J10.2 (Pin_2)
- new net GP.GPIO10: J10.10 (Pin_10)
Changed lines of the file:
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@@
 	(wire
 		(pts
-			(xy 193.04 87.63) (xy 205.74 87.63)
-		)
-		(stroke
-			(width 0)
-			(type default)
-		)
-	)
-	(wire
-		(pts
 			(xy 115.57 137.16) (xy 115.57 138.43)
 		)
@@
 	(wire
 		(pts
+			(xy 193.04 87.63) (xy 205.74 87.63)
+		)
+		(stroke
+			(width 0)
+			(type default)
+		)
+	)
+	(wire
+		(pts
 			(xy 193.04 77.47) (xy 205.74 77.47)
 		)
@@
 	(wire
 		(pts
+			(xy 193.04 90.17) (xy 205.74 90.17)
+		)
+		(stroke
+			(width 0)
+			(type default)
+		)
+	)
+	(wire
+		(pts
 			(xy 110.49 58.42) (xy 124.46 58.42)
 		)
@@
 	(wire
 		(pts
-			(xy 193.04 90.17) (xy 205.74 90.17)
-		)
-		(stroke
-			(width 0)
-			(type default)
-		)
-	)
-	(wire
-		(pts
 			(xy 193.04 72.39) (xy 205.74 72.39)
 		)
@@
 		)
 	)
-	(label "GP.SDA"
-		(at 193.04 59.69 0)
-		(effects
-			(font
-				(size 1.27 1.27)
-			)
-			(justify left bottom)
-		)
-	)
 	(label "LED.SUCCESS"
 		(at 109.22 101.6 180)
@@
 	)
 	(label "GP.GPIO13"
-		(at 193.04 80.01 0)
+		(at 193.04 77.47 0)
 		(effects
 			(font
@@
 		)
 	)
-	(label "GP.GPIO38"
-		(at 193.04 82.55 0)
+	(label "GP.GPIO10"
+		(at 193.04 80.01 0)
 		(effects
 			(font
@@
 		)
 	)
+	(label "GP.SCL"
+		(at 193.04 87.63 0)
+		(effects
+			(font
+				(size 1.27 1.27)
+			)
+			(justify left bottom)
+		)
+	)
+	(label "GP.GPIO_A_2"
+		(at 193.04 62.23 0)
+		(effects
+			(font
+				(size 1.27 1.27)
+			)
+			(justify left bottom)
+		)
+	)
 	(label "GP.GPIO12"
 		(at 124.46 74.93 180)
@@
 	)
 	(label "GP.GPIO12"
-		(at 193.04 77.47 0)
+		(at 193.04 82.55 0)
 		(effects
 			(font
@@
 		)
 	)
-	(label "GP.GPIO_A_1"
-		(at 193.04 87.63 0)
-		(effects
-			(font
-				(size 1.27 1.27)
-			)
-			(justify left bottom)
-		)
-	)
 	(label "GP.D-"
 		(at 93.98 52.07 180)
@@
 		)
 	)
+	(label "GP.GPIO_A_1"
+		(at 193.04 59.69 0)
+		(effects
+			(font
+				(size 1.27 1.27)
+			)
+			(justify left bottom)
+		)
+	)
 	(label "GP.MISO"
 		(at 193.04 69.85 0)
@@
 	)
 	(label "GP.SDA"
+		(at 193.04 90.17 0)
+		(effects
+			(font
+				(size 1.27 1.27)
+			)
+			(justify left bottom)
+		)
+	)
+	(label "GP.SDA"
 		(at 124.46 49.53 180)
 		(effects
@@
 		)
 	)
-	(label "GP.GPIO_A_2"
-		(at 193.04 90.17 0)
-		(effects
-			(font
-				(size 1.27 1.27)
-			)
-			(justify left bottom)
-		)
-	)
-	(label "GP.SCL"
-		(at 193.04 62.23 0)
-		(effects
-			(font
-				(size 1.27 1.27)
-			)
-			(justify left bottom)
-		)
-	)
 	(hierarchical_label "GP{USB}"
 		(shape input)
@@
 		(lib_name "+BATT_1")
 		(lib_id "power:+BATT")
-		(at 160.02 55.88 0)
+		(at 160.02 66.04 0)
 		(unit 1)
 		(body_style 1)
@@
 		(fields_autoplaced yes)
 		(property "Reference" "#PWR017"
-			(at 160.02 59.69 0)
+			(at 160.02 69.85 0)
 			(hide yes)
 			(show_name no)
@@
 		)
 		(property "Value" "+BATT"
-			(at 157.48 54.6099 0)
+			(at 157.48 64.7699 0)
 			(show_name no)
 			(do_not_autoplace no)
@@
 		)
 		(property "Footprint" ""
-			(at 160.02 55.88 0)
+			(at 160.02 66.04 0)
 			(hide yes)
 			(show_name no)
@@
 		)
 		(property "Datasheet" ""
-			(at 160.02 55.88 0)
+			(at 160.02 66.04 0)
 			(hide yes)
 			(show_name no)
@@
 		)
 		(property "Description" ""
-			(at 160.02 55.88 0)
+			(at 160.02 66.04 0)
 			(hide yes)
 			(show_name no)
@@
 	(symbol
 		(lib_id "power:+3.3V")
-		(at 160.02 66.04 0)
+		(at 160.02 55.88 0)
 		(mirror y)
 		(unit 1)
@@
 		(fields_autoplaced yes)
 		(property "Reference" "#PWR053"
-			(at 160.02 69.85 0)
+			(at 160.02 59.69 0)
 			(hide yes)
 			(show_name no)
@@
 		)
 		(property "Value" "+3.3V"
-			(at 157.48 64.7699 0)
+			(at 157.48 54.6099 0)
 			(show_name no)
 			(do_not_autoplace no)
@@
 		)
 		(property "Footprint" ""
-			(at 160.02 66.04 0)
+			(at 160.02 55.88 0)
 			(hide yes)
 			(show_name no)
@@
 		)
 		(property "Datasheet" ""
-			(at 160.02 66.04 0)
+			(at 160.02 55.88 0)
 			(hide yes)
 			(show_name no)
@@
 		)
 		(property "Description" ""
-			(at 160.02 66.04 0)
+			(at 160.02 55.88 0)
 			(hide yes)
 			(show_name no)
